Commit message: Update Description and create omni_drive and gazebo

File: src/omni_carver_description/urdf/robot/base.xacro (robot description, xacro)
@@ -1,5 +1,5 @@
 <?xml version='1.0' encoding='utf-8'?>
 <robot xmlns:xacro="http://www.ros.org/wiki/xacro">
-    <xacro:include filename="$(find twheel_description)/urdf/properties.xacro"/>
+    <xacro:include filename="$(find omni_carver_description)/urdf/robot/properties.xacro"/>
     <xacro:macro name="base" params="path">
         <link name="base_footprint"/>

File: src/omni_carver_description/urdf/robot/castor.xacro (robot description, xacro)
@@ -1,5 +1,5 @@
 <?xml version='1.0' encoding='utf-8'?>
 <robot xmlns:xacro="http://www.ros.org/wiki/xacro">
-  <xacro:include filename="$(find twheel_description)/urdf/properties.xacro"/>
+  <xacro:include filename="$(find omni_carver_description)/urdf/robot/properties.xacro"/>
   <xacro:macro name="castor" params="name translation_x translation_y">
     <link name="${name}_castor">

File: src/omni_carver_description/urdf/robot/properties.xacro (robot description, xacro)
@@ -1,6 +1,6 @@
 <?xml version='1.0' encoding='utf-8'?>
 <robot xmlns:xacro="http://www.ros.org/wiki/xacro">
-  <xacro:property name="params_path" value="$(find xxx_description)/config/properties.yaml"/> <!-- Need seperate property for xacro inorder processing -->
-  <xacro:property name="mp" value="${load_yaml(params_path)}"/> <!-- Read in the yaml dict as mp (short for model parameters) -->
+  <xacro:property name="params_path" value="$(find omni_carver_description)/config/properties.yaml"/> <!-- Need seperate property for xacro inorder processing -->
+  <xacro:property name="mp" value="${xacro.load_yaml(params_path)}"/> <!-- Read in the yaml dict as mp (short for model parameters) -->
   <!-- Mathematics Constants -->
   <xacro:property name="PI" value="3.1415926535897931"/>
@@ -15,5 +15,5 @@
   <xacro:property name="BASE_HEIGHT" value="${mp['base_height']}"/>
   <xacro:property name="BASE_ELEVATION" value="${mp['base_elevation']}"/>
-  <xacro:property name="PACKAGE_NAME" value="xxx_description"/>
+  <xacro:property name="PACKAGE_NAME" value="omni_carver_description"/>
   <xacro:property name="BASE_MESH_PATH" value="${mp['base_mesh_path']}"/>
   <xacro:property name="BASE_MESH_Z_OFFSET" value="${mp['base_mesh_z_offset']}"/>
@@ -37,3 +37,34 @@
   <xacro:property name="CAMERA_OFFSET" value="${mp['camera_offset']}"/>
   <xacro:property name="CAMERA_HEIGHT" value="${mp['camera_height']}"/>
+  <!-- Base Inertial Properties -->
+  <xacro:property name="BASE_M" value="40.0"/>
+  <xacro:property name="BASE_COM" value="0.0002 0.0001 -0.0001"/>
+  <xacro:property name="BASE_Ixx" value="1.79366667"/>
+  <xacro:property name="BASE_Iyy" value="1.28666667"/>
+  <xacro:property name="BASE_Izz" value="0.230966667"/>
+  <xacro:property name="BASE_Ixy" value="0"/>
+  <xacro:property name="BASE_Ixz" value="0"/>
+  <xacro:property name="BASE_Iyz" value="0"/>
+  <!-- Wheel Inertial Properties -->
+  <xacro:property name="WHEEL_M" value="2.9"/>
+  <xacro:property name="WHEEL_COM" value="0 0 0"/>
+  <xacro:property name="WHEEL_Ixx" value="0.00564437"/>
+  <xacro:property name="WHEEL_Iyy" value="0.00564437"/>
+  <xacro:property name="WHEEL_Izz" value="0.01047625"/>
+  <xacro:property name="WHEEL_Ixy" value="0"/>
+  <xacro:property name="WHEEL_Ixz" value="0"/>
+  <xacro:property name="WHEEL_Iyz" value="0"/>
+  <!-- Castor Inertial Properties -->
+  <xacro:property name="CASTOR_M" value="0.2"/>
+  <xacro:property name="CASTOR_COM" value="0 0 0"/>
+  <xacro:property name="CASTOR_Ixx" value="0.00004437"/>
+  <xacro:property name="CASTOR_Iyy" value="0.00004437"/>
+  <xacro:property name="CASTOR_Izz" value="0.00047625"/>
+  <xacro:property name="CASTOR_Ixy" value="0"/>
+  <xacro:property name="CASTOR_Ixz" value="0"/>
+  <xacro:property name="CASTOR_Iyz" value="0"/>
+  <!-- Joint Properties -->
+  <xacro:property name="U_MAX" value="300"/>
+  <xacro:property name="V_MAX" value="300"/>
+  <xacro:property name="WHEEL_JOINT_DAMP" value="0"/>
 </robot>

File: src/omni_carver_description/urdf/robot/sensor.xacro (robot description, xacro)
@@ -1,5 +1,5 @@
 <?xml version='1.0' encoding='utf-8'?>
 <robot xmlns:xacro="http://www.ros.org/wiki/xacro">
-  <xacro:include filename="$(find twheel_description)/urdf/properties.xacro"/>
+  <xacro:include filename="$(find omni_carver_description)/urdf/robot/properties.xacro"/>
   <!-- Contents-->
   <xacro:macro name="sensor_link" params="">

File: src/omni_carver_description/urdf/robot/twheel.urdf (robot description, URDF)
Before this commit: robot twheel_bot, 6 links, 5 joints
Links:
- link base_link: geometry visual mesh filename=package://omni_carver_description/meshes/twheel_base.STL

File: src/omni_carver_description/urdf/robot/twheel.xacro (robot description, xacro)
@@ -1,5 +1,5 @@
 <?xml version='1.0' encoding='utf-8'?>
-<robot xmlns:xacro="http://www.ros.org/wiki/xacro" name="twheel">
-  <xacro:include filename="$(find twheel_description)/urdf/twheel.xacro"/>
+<robot xmlns:xacro="http://www.ros.org/wiki/xacro" name="omni_carver">
+  <xacro:include filename="$(find omni_carver_description)/urdf/robot/twheel.xacro"/>
   <xacro:include filename="$(find twheel_gazebo)/urdf/graphics.gazebo.xacro"/>
   <xacro:include filename="$(find twheel_gazebo)/urdf/sensor.gazebo.xacro"/>

File: src/omni_carver_description/urdf/robot/twheel_backup.urdf (robot description, URDF)
Before this commit: robot twheel, 4 links, 3 joints
Links:
- link base_link: geometry visual mesh filename=package://omni_carver_description/meshes/coconut.stl

File: src/omni_carver_description/urdf/robot/twheel_gazebo.xacro (robot description, xacro)
@@ -1,9 +1,9 @@
 <?xml version='1.0' encoding='utf-8'?>
-<robot xmlns:xacro="http://www.ros.org/wiki/xacro" name="twheel">
-    <xacro:include filename="$(find twheel_description)/urdf/properties.xacro"/>
-    <xacro:include filename="$(find twheel_description)/urdf/base.xacro"/>
-    <xacro:include filename="$(find twheel_description)/urdf/wheel.xacro"/>
-    <xacro:include filename="$(find twheel_description)/urdf/castor.xacro"/>
-    <xacro:include filename="$(find twheel_description)/urdf/sensor.xacro"/>
+<robot xmlns:xacro="http://www.ros.org/wiki/xacro" name="omni_carver">
+    <xacro:include filename="$(find omni_carver_description)/urdf/robot/properties.xacro"/>
+    <xacro:include filename="$(find omni_carver_description)/urdf/robot/base.xacro"/>
+    <xacro:include filename="$(find omni_carver_description)/urdf/robot/wheel.xacro"/>
+    <xacro:include filename="$(find omni_carver_description)/urdf/robot/castor.xacro"/>
+    <xacro:include filename="$(find omni_carver_description)/urdf/robot/sensor.xacro"/>
     <xacro:base path="$(find ${PACKAGE_NAME})/${BASE_MESH_PATH}"/>
     <xacro:wheel name="left" translation_y="${WHEEL_SEPARATION/2}"/>

File: src/omni_carver_description/urdf/robot/wheel.xacro (robot description, xacro)
@@ -1,5 +1,5 @@
 <?xml version='1.0' encoding='utf-8'?>
-<robot xmlns:xacro="http://www.ros.org/wiki/xacro" name="twheel">
-    <xacro:include filename="$(find twheel_description)/urdf/properties.xacro"/>
+<robot xmlns:xacro="http://www.ros.org/wiki/xacro" name="omni_carver">
+    <xacro:include filename="$(find omni_carver_description)/urdf/robot/properties.xacro"/>
     <xacro:macro name="wheel" params="name translation_y">
         <link name="${name}_wheel">
