Commit message: Update controller, urdf, and kinematic

File: src/omni_carver_description/xacro/gazebo_control.xacro (robot description, xacro)
@@ -6,8 +6,17 @@
           <plugin>gz_ros2_control/GazeboSimSystem</plugin>
       </hardware>
+      <joint name="rim_right_joint">
+        <command_interface name="velocity">
+          <param name="min">-10</param>
+          <param name="max">10</param>
+        </command_interface>
+        <state_interface name="position"/>
+        <state_interface name="velocity"/>
+        <state_interface name="effort"/>
+      </joint>
       <joint name="rim_left_joint">
         <command_interface name="velocity">
-          <param name="min">-5</param>
-          <param name="max">5</param>
+          <param name="min">-10</param>
+          <param name="max">10</param>
         </command_interface>
         <state_interface name="position"/>
@@ -17,15 +26,6 @@
       <joint name="rim_back_joint">
         <command_interface name="velocity">
-          <param name="min">-5</param>
-          <param name="max">5</param>
-        </command_interface>
-        <state_interface name="position"/>
-        <state_interface name="velocity"/>
-        <state_interface name="effort"/>
-      </joint>
-      <joint name="rim_right_joint">
-        <command_interface name="velocity">
-          <param name="min">-5</param>
-          <param name="max">5</param>
+          <param name="min">-10</param>
+          <param name="max">10</param>
         </command_interface>
         <state_interface name="position"/>

File: src/omni_carver_description/xacro/main.urdf.xacro (robot description, xacro)
@@ -12,5 +12,6 @@
 	<link name="base_link">
 	<inertial>
-		<mass value="0.07862944645"/>
+		<!-- <mass value="0.07862944645"/> -->
+		<mass value="2"/>
 		<inertia
 			ixx="0.00002035985530754"
@@ -85,8 +86,4 @@
 				name="gz::sim::systems::Imu">
 		</plugin>
-		<!-- <plugin
-			filename="gz-sim-physics-system"
-			name="gz::sim::systems::Physics">
-		</plugin> -->
 	</gazebo>
 </robot>

File: src/omni_carver_description/xacro/rim.urdf.xacro (robot description, xacro)
@@ -9,5 +9,6 @@
 			<inertial>
 				<origin xyz="0 0 -0.000343" />
-				<mass value="0.00835758" />
+				<!-- <mass value="0.00835758" /> -->
+				<mass value="1.0" />
 				<inertia
 					ixx="6.63684e-07"

File: src/omni_carver_description/xacro/roller.urdf.xacro (robot description, xacro)
@@ -7,5 +7,5 @@
 		<link name="roller_${name}_rim_${parent}_link">
 			<inertial>
-				<mass value="0.00113845"/>
+				<mass value="0.5"/>
 				<inertia
 					ixx="2.53776e-08"
