Commit message: Update Firmware and Connect with pyserial

File: src/omni_carver_description/gazebo_description/lidar.xacro (robot description, xacro)
@@ -30,5 +30,5 @@
       <sensor name="laser" type="gpu_lidar">
         <gz_frame_id>laser_link</gz_frame_id>
-        <topic>scan</topic>
+        <topic>/scan</topic>
         <update_rate>10</update_rate>
         <lidar>
@@ -46,5 +46,5 @@
             <resolution>0.01</resolution>
           </range>
-          <frame_id>/laser_link</frame_id>
+          <frame_id>laser_link</frame_id>
         </lidar>
         <alwaysOn>ture</alwaysOn>

File: src/omni_carver_description/gazebo_description/main.urdf.xacro (robot description, xacro)
@@ -4,10 +4,17 @@
 	name="open_base"
 >
-	<xacro:include filename="$(find omni_carver_description)/xacro/rim.urdf.xacro"/>
-	<xacro:include filename="$(find omni_carver_description)/xacro/gazebo_control.xacro"/>
-	<xacro:include filename="$(find omni_carver_description)/xacro/inertial_macros.xacro"/>
-	<xacro:include filename="$(find omni_carver_description)/xacro/lidar.xacro"/>
-	<xacro:include filename="$(find omni_carver_description)/xacro/imu.xacro"/>
+	<xacro:include filename="$(find omni_carver_description)/gazebo_description/rim.urdf.xacro"/>
+	<xacro:include filename="$(find omni_carver_description)/gazebo_description/gazebo_control.xacro"/>
+	<xacro:include filename="$(find omni_carver_description)/gazebo_description/inertial_macros.xacro"/>
+	<xacro:include filename="$(find omni_carver_description)/gazebo_description/lidar.xacro"/>
+	<xacro:include filename="$(find omni_carver_description)/gazebo_description/imu.xacro"/>
 	<link name="origin_link"/>
+	<joint name="base_footprint_joint" type="fixed">
+		<origin xyz="0 0 0" rpy="0 0 0"/>
+		<parent link="origin_link"/>
+		<child link="base_footprint"/>
+	</joint>
+	<link name="base_footprint">
+	</link>
 	<link name="base_link">
 	<inertial>

File: src/omni_carver_description/gazebo_description/rim.urdf.xacro (robot description, xacro)
@@ -1,5 +1,5 @@
 <?xml version="1.0"?>
 <robot xmlns:xacro="http://www.ros.org/wiki/xacro">
-	<xacro:include filename="$(find omni_carver_description)/xacro/roller.urdf.xacro" />
+	<xacro:include filename="$(find omni_carver_description)/gazebo_description/roller.urdf.xacro" />
 	<xacro:macro
 		name="rim_macro"
@@ -29,10 +29,8 @@
 			</visual>
 			<collision>
-				<attach_mesh_shape_feature>true</attach_mesh_shape_feature>
 				<geometry>
 					<mesh filename="package://omni_carver_description/mesh/rim.stl">
 					</mesh>
 				</geometry>
-				<attach_mesh_shape_feature>true</attach_mesh_shape_feature>
 			</collision>
 		</link>

File: src/omni_carver_description/gazebo_description/roller.urdf.xacro (robot description, xacro)
@@ -26,10 +26,8 @@
 			</visual>
 			<collision>
-				<attach_mesh_shape_feature>true</attach_mesh_shape_feature>
 				<geometry>
 					<mesh filename="package://omni_carver_description/mesh/roller.stl">
 					</mesh>
 				</geometry>
-				<attach_mesh_shape_feature>true</attach_mesh_shape_feature>
 			</collision>
 		</link>
